File: Hardware/ECG_BOB/pc_ads1292r_brk_v3.sch (EAGLE design)
At the start: 63 parts, among them Q1 BSS138, Q2 BSS138, Q3 BSS138, Q4 BSS138, Q5 BSS138, Q6 BSS138, Q7 BSS138

Commit message: added new design file
Parts:
- removed C58: DNP, rcl:C-EUC0402
- removed Q1, Q2, Q3, Q4, Q5, Q6, Q7: BSS138, SparkFun:MOSFET-NCHANNELSMD
- removed R1, R11, R13, R14, R17, R2, R25, R26, R4, R5, R6, R7, R8, R9: 10K, SparkFun:RESISTOR0603-RES
- added C2: 100n, rcl:C-EUC0402
- added LOGO1: OSHW_LOGO_FILLX0100-NT, ohw-logo:OSHW_LOGO_FILLX0100-NT
- added U1: (no value), adafruit:TXB0108PWR
- C1: value (none) -> 100n
- U$8: value (none) -> ADS1292R-TQFP; device circuitects:ADS1292RPVQFN32 -> circuitects:ADS1292R-TQFP
Connections:
- net !ADS_DRDY: now also U1.A1; no longer Q3.S, R2.2
- net !ARD_DRDY: now also U1.B1; no longer Q3.D, R5.2
- net +3V3: now also C2.2, U1.OE, U1.VCCA; no longer Q1.G, Q2.G, Q3.G, Q4.G, Q5.G, Q6.G, Q7.G, R1.1, R11.1, R14.1, R2.1, R25.1, R6.1, R8.1
- net +5V: now also C1.2, U1.VCCB
- net ADS_PWDN: now also U1.A7; no longer Q1.S, R1.2
- net ADS_START: now also U1.A6; no longer Q2.S, R6.2
- net ARD_CS0: now also U1.B5; no longer Q7.D, R26.2
- net ARD_MISO: now also U1.B2; no longer Q5.D, R13.2
- net ARD_MOSI: now also U1.B4; no longer Q4.D, R9.2
- net ARD_PWDN: now also U1.B7; no longer Q1.D, R4.2
- net ARD_SCK: now also U1.B3; no longer Q6.D, R17.2
- net ARD_START: now also U1.B6; no longer Q2.D, R7.2
- net GND: now also C1.1, C2.1, U1.GND; no longer C1.2, C58.1
- net N$30: now also JP3.LEFT; no longer C1.1, JP3.RIGHT
- net N$45: now also JP3.RIGHT; no longer C58.2, JP3.SLEEVE
- net N$51: now also JP3.SLEEVE; no longer JP3.LEFT
- net SPI_CS0: now also U1.A5; no longer Q7.S, R25.2
- net SPI_MISO: now also U1.A2; no longer Q5.S, R11.2
- net SPI_MOSI: now also U1.A4; no longer Q4.S, R8.2
- net SPI_SCK: now also U1.A3; no longer Q6.S, R14.2
- net VCC: no longer R13.1, R17.1, R26.1, R4.1, R5.1, R7.1, R9.1
Other:
- note removed: "Channel 1"
- note removed: "Channel 2"
- note removed: "Channel 3"
- note removed: "Channel 4"
- note removed: "Channel 5"
- note removed: "Channel 6"
- note removed: "Channel 7"

Commit message: Add files via upload
Parts:
- removed C39: 10n, rcl:C-EUC0402
- removed U$13: TPS717XX, circuitects:TPS717XX
- added U$1: PROTY-LOGO, circuitects:PROTY-LOGO
- added U2: AP2112K-3.3V, SparkFun-PowerIC:V_REG_LDOSMD
Connections:
- removed net N$1: C39.2, U$13.FB
- net +3V3: now also U2.OUT; no longer U$13.OUT
- net +5V: now also U2.EN, U2.IN; no longer C1.2, U$13.EN, U$13.IN, U1.VCCB
- net GND: now also U2.GND; no longer C39.1, U$13.GND
- net VCC: now also C1.2, U1.VCCB
Other:
- note added: "CONNECTOR"
- note added: "LOGIC LEVEL CONVERTER"
- note added: "POWER SUPPLY"
